File: Power - Sequencing.kicad_sch (KiCad schematic)
At the start: 0 parts

Commit message: First draft of the schematic
Other:
- title: Power - Sequencing -> MCU
Changed lines of the file:
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@@
 	(paper "A4")
 	(title_block
-		(title "Power - Sequencing")
+		(title "MCU")
 		(date "2025-01-12")
 		(rev "${REVISION}")
