File: IndustrialSense.kicad_pcb (KiCad board)
At the start: 4 copper layers, 46.9 x 90 mm, 120 parts, among them CN2 B4B-ZR (LF)(SN), CN3 ZH1.5-6P-LT, CN4 B4B-ZR (LF)(SN), J5 Conn_01x10_Socket, J6 Conn_01x10_Socket, Q1 SISA14DN-T1-GE3, Q13 MMBT3904, Q15 LMBT3904DW1T1G, Q2 SISA14DN-T1-GE3, Q3 SISA14DN-T1-GE3, Q4 SISA14DN-T1-GE3, Q5 CEM4435A, Q6 CH221K, SW2 SKRKAEE020, SW3 SKRKAEE020, U1 ESP32-S3-WROOM-1U-N16, U10 LM74700QDBVRQ1, U11 CN3795, U12 XFL4020-222MEC_C122469, U13 B6B-ZR (LF)(SN), U14 CH334F, U15 TPS3831G33DQNR, U17 THVD1406DR, U2 B6B-ZR (LF)(SN), U3 CH343P, U4 MAX17049G+T10, U5 LM74700QDBVRQ1, U6 LM74700QDBVRQ1, U7 TPS62132RGTT, U8 LM74700QDBVRQ1, U9 XC6209F332MR-G, X1 X322512MSB4SI

Commit message: [PCB] Checked
Parts:
- moved TP3 21.5 mm to (148.9, 100.3)
- moved D10 0.50 mm to (159.8, 130.0)
- moved R67 0.50 mm to (160.6, 124.5)
- moved R68 0.50 mm to (159.1, 124.5)
- moved R69 0.50 mm to (159.8, 127.0)
Routing:
- net Net-(U17-B): track 3.21 -> 2.54 mm
- net /Project Architecture/External Connectors/RS485_A: track 9.12 -> 9.62 mm
- net Net-(U17-A): track 3.07 -> 2.56 mm
- net GND: vias 93 -> 157
Other:
- board text added: "BATT"
- board text added: "BTN"
- board text added: "EXT USB"
- board text added: "I2C"
- board text added: "LTE"
- board text added: "MISC"
- board text added: "RGB"
- board text added: "RS485"
- board text added: "SOLAR"
- board text added: "TP1"
- board text added: "TP10"
- board text added: "TP2"
- board text added: "TP3"
- board text added: "TP4"
- board text added: "TP5"
- board text added: "TP6"
- board text added: "TP7"
- board text added: "TP8"
- board text added: "TP9"
- board text added: "USB"
- board text added: "µSD"

Commit message: [PCB][Added] Gerber, CPL, BOM ready
Parts:
- C1: value 47uF -> 47u
- C7: value 10u -> 47u

Commit message: Update Outputs (release)
Other:
- board text added: "0.02mm"
- board text added: "0.035mm (1.00oz)"
- board text added: "0.07mm (2.00oz)"
- board text added: "0.1mm"
- board text added: "0.75mm"
- board text added: "B.Mask"
- board text added: "B.Paste"
- board text added: "B.Silkscreen"
- board text added: "Copper"
- board text added: "Copper Layer"
- board text added: "Core"
- board text added: "Dielectric"
- board text added: "Direct Printing"
- board text added: "F.Mask"
- board text added: "F.Paste"
- board text added: "F.Silkscreen"
- board text added: "FR4"
- board text added: "FR4_7628"
- board text added: "GBR"
- board text added: "Gerber"
- board text added: "L1"
- board text added: "L2"
- board text added: "L3"
- board text added: "L4"
- board text added: "Layer"
- board text added: "Legend"
- board text added: "Material"
- board text added: "Note: external layer thicknesses are specified after plating"
- board text added: "Paste Mask"
- board text added: "Prepreg"
- board text added: "Signal"
- board text added: "Solder Mask"
- board text added: "Solder Resist"
- board text added: "Thickness"
- board text added: "Total thickness: 1.2mm"
- board text added: "Type"
